File: HilBox_Interfaces.kicad_sch (KiCad schematic)
At the start: 16 parts, among them U27 TJA1051T-3, U28 MAX3485

Commit message: Layout 90% done
Parts:
- R82, R83: footprint Resistor_SMD:R_0603_1608Metric -> Resistor_SMD:R_1206_3216Metric; JLC_PN C23162 -> C1469
Changed lines of the file:
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@@
 			)
 		)
-		(property "Footprint" "Resistor_SMD:R_0603_1608Metric"
+		(property "Footprint" "Resistor_SMD:R_1206_3216Metric"
 			(at 76.2 54.102 90)
 			(effects
@@
 			)
 		)
-		(property "JLC_PN" "C23162"
+		(property "JLC_PN" "C1469"
 			(at 76.2 55.88 90)
 			(effects
@@
 			)
 		)
-		(property "Footprint" "Resistor_SMD:R_0603_1608Metric"
+		(property "Footprint" "Resistor_SMD:R_1206_3216Metric"
 			(at 76.2 49.022 90)
 			(effects
@@
 			)
 		)
-		(property "JLC_PN" "C23162"
+		(property "JLC_PN" "C1469"
 			(at 76.2 50.8 90)
 			(effects
