File: HilBox.kicad_pcb (KiCad board)
At the start: 4 copper layers, 172.1 x 119.7 mm, 274 parts, among them J1 Conn_01x02_Pin, J11 Conn_01x03_Pin, J13 Conn_01x10_Pin, J17 USB_C_Plug_USB2.0, J2 Conn_01x02_Pin, J20 Conn_01x04_Pin, J21 Conn_01x02_Pin, J22 Conn_01x02_Pin, J23 Conn_01x02_Pin, J24 Conn_01x06_Pin, J3 Conn_01x02_Pin, J4 Conn_01x02_Pin, J9 Conn_01x10_Pin, K1 G5NB, K2 G5NB, K3 G5NB, K4 G5NB, K5 G5NB, Q10 BC847BS, Q11 BC847BS, Q12 BC847BS, Q22 BC847BS, Q24 BC847BS, Q8 BC847BS, Q9 BC847BS, U1 STM32F407VGTx, U2 MCP4822, U24 TLV272IS-13, U25 FT232RL, U27 TJA1051T-3, U28 MAX3485, U29 LM5007MM, U3 BU4S66G2-TR, U30 LM5007MM, U31 LM5007MM, U32 USB6B1RL, U5 BU4S66G2-TR, U6 MCP4822, U7 TLV272IS-13, U8 BU4S66G2-TR, U9 BU4S66G2-TR, Y1 20MHz

Commit message: Modification in half of target
Parts:
- removed D22, D24: RED, LED_SMD:LED_1206_3216Metric
- removed D23, D25: US1A, Diode_SMD:D_SMA
- removed D41: FM407, Diode_SMD:D_SMA
- removed J1, J2, J3, J4: Conn_01x02_Pin, Connector_PinHeader_2.54mm:PinHeader_1x02_P2.54mm_Vertical
- removed J9: Conn_01x10_Pin, Gascard_Lib:Terminal_Block_3_81_10p
- removed K2, K3, K4, K5: G5NB, Relay_THT:Relay_SPST_Omron_G5NB
- removed Q11, Q12: BC847BS, Package_TO_SOT_SMD:SOT-363_SC-70-6
- removed R126: 220R, Resistor_SMD:R_0402_1005Metric
- removed R179, R182, R74, R77: 10k, Resistor_SMD:R_0603_1608Metric
- removed R180, R181, R73, R76: 2k2, Resistor_SMD:R_0603_1608Metric
- removed R75, R78: 680R, Resistor_SMD:R_0603_1608Metric
- removed R79, R80: 470k, Resistor_SMD:R_1206_3216Metric
- added C13: 1n/2kV, Capacitor_SMD:C_1206_3216Metric, F.Cu at (-45.3, 96.5)
- added C14: 100n/25V, Capacitor_SMD:C_0402_1005Metric, F.Cu at (-60.1, 89.2)
- added C15: 100n/25V, Capacitor_SMD:C_0402_1005Metric, F.Cu at (-60.1, 91.2)
- added C16: 100n/25V, Capacitor_SMD:C_0402_1005Metric, F.Cu at (-60.1, 93.2)
- added C17: 100n/25V, Capacitor_SMD:C_0402_1005Metric, F.Cu at (-60.1, 95.2)
- added C18: 100n/25V, Capacitor_SMD:C_0402_1005Metric, F.Cu at (-60.1, 97.1)
- added C19: 100n/25V, Capacitor_SMD:C_0402_1005Metric, F.Cu at (-60.1, 99.1)
- added C20: 100n/25V, Capacitor_SMD:C_0402_1005Metric, F.Cu at (-60.1, 101.1)
- added C21: 4u7/10V, Capacitor_SMD:C_0402_1005Metric, F.Cu at (-60.1, 103.0)
- added D10: LED BLUE, LED_SMD:LED_0603_1608Metric, F.Cu at (-18.4, 70.6)
- added D11: LED BLUE, LED_SMD:LED_0603_1608Metric, F.Cu at (-18.4, 73.2)
- added D12: LED_RGBA, Relays:RELAY_G6K-2F_DC5, F.Cu at (154.8, 45.0)
- added D5: BLUE, LED_SMD:LED_0603_1608Metric, F.Cu at (-42.0, 101.6)
- added D6: WHITE, LED_SMD:LED_0603_1608Metric, F.Cu at (-42.0, 104.2)
- added D7: LED YELLOW, LED_SMD:LED_0603_1608Metric, F.Cu at (-18.4, 62.8)
- added D8: LED GREEN, LED_SMD:LED_0603_1608Metric, F.Cu at (-18.4, 65.4)
- added D9: LED BLUE, LED_SMD:LED_0603_1608Metric, F.Cu at (-18.4, 68.0)
- added J7: USB_C_Plug_USB2.0, Connector_USB:USB_C_Receptacle_GCT_USB4105-xx-A_16P_TopMnt_Horizontal, F.Cu at (151.8, 114.0)
- added J8: Conn_01x04_Pin, Connector_PinHeader_2.54mm:PinHeader_1x04_P2.54mm_Vertical, F.Cu at (144.0, 111.4)
- added R15: 1M, Resistor_SMD:R_0603_1608Metric, F.Cu at (-63.5, 89.5)
- added R16: 5k1, Resistor_SMD:R_0603_1608Metric, F.Cu at (-63.5, 92.0)
- added R17: 5k1, Resistor_SMD:R_0603_1608Metric, F.Cu at (-63.5, 94.5)
- added R19: 22R/1%, Resistor_SMD:R_0402_1005Metric, F.Cu at (-45.5, 101.3)
- added R20: 0R/1%, Resistor_SMD:R_0603_1608Metric, F.Cu at (-63.5, 97.0)
- added R21: 22R/1%, Resistor_SMD:R_0402_1005Metric, F.Cu at (-45.5, 103.3)
- added R22: 10k/02, Resistor_SMD:R_0402_1005Metric, F.Cu at (-45.5, 105.3)
- added R23: 680R, Resistor_SMD:R_0603_1608Metric, F.Cu at (-63.5, 99.6)
- added R24: 0R/1%, Resistor_SMD:R_0603_1608Metric, F.Cu at (-63.5, 102.1)
- added R25: 0R/1%, Resistor_SMD:R_0603_1608Metric, F.Cu at (-63.5, 104.6)
- added R26: 680R, Resistor_SMD:R_0603_1608Metric, F.Cu at (-63.5, 107.1)
- added R27: 680R, Resistor_SMD:R_0603_1608Metric, F.Cu at (-14.4, 62.8)
- added R28: 680R, Resistor_SMD:R_0603_1608Metric, F.Cu at (-14.4, 65.3)
- added R29: 680R, Resistor_SMD:R_0603_1608Metric, F.Cu at (-14.4, 67.8)
- added R30: 680R, Resistor_SMD:R_0603_1608Metric, F.Cu at (-14.4, 70.3)
- added R31: 680R, Resistor_SMD:R_0603_1608Metric, F.Cu at (-14.4, 72.8)
- added R32: 100R, Resistor_SMD:R_0603_1608Metric, F.Cu at (-10.4, 62.8)
- added R33: 100R, Resistor_SMD:R_0603_1608Metric, F.Cu at (-10.4, 65.3)
- added R34: 100R, Resistor_SMD:R_0603_1608Metric, F.Cu at (-10.4, 67.8)
- added R35: 100R, Resistor_SMD:R_0603_1608Metric, F.Cu at (-10.4, 70.3)
- added R36: 100R, Resistor_SMD:R_0603_1608Metric, F.Cu at (-10.4, 72.8)
- added R37: 100R, Resistor_SMD:R_0603_1608Metric, F.Cu at (-6.42, 62.8)
- added R38: 330R, Resistor_SMD:R_0603_1608Metric, F.Cu at (-6.42, 65.3)
- added R39: 330R, Resistor_SMD:R_0603_1608Metric, F.Cu at (-6.42, 67.8)
- added R40: 680R, Resistor_SMD:R_0603_1608Metric, F.Cu at (-6.42, 70.3)
- added SW1: SW_DIP_x06, Button_Switch_SMD:SW_DIP_SPSTx06_Slide_6.7x16.8mm_W8.61mm_P2.54mm_LowProfile, F.Cu at (127.0, 83.2)
- added U11: USB6B1RL, Package_SO:SOIC-8_3.9x4.9mm_P1.27mm, F.Cu at (-43.9, 91.6)
- added U12: FT232RL, Package_SO:SSOP-28_5.3x10.2mm_P0.65mm, F.Cu at (165.2, 111.6)
- D32: value YELLOW -> RED
- D33: value PURPLE -> RED
- D34: value AMBER -> RED
- J13: footprint Gascard_Lib:Terminal_Block_3_81_10p -> Connector_Phoenix_MC:PhoenixContact_MCV_1,5_10-G-3.81_1x10_P3.81mm_Vertical
- K1: value G5NB -> G6K-2F-Y-5V; footprint Relay_THT:Relay_SPST_Omron_G5NB -> Relays:RELAY_G6K-2F_DC5
- R125, R166: value 220R -> 680R
- moved C11 78.3 mm to (2.85, 68.3), turned to 90 degrees
- moved R187 76.7 mm to (0.60, 74.8), turned to 180 degrees
- moved D4 75.9 mm to (5.40, 67.4), turned to 90 degrees
- moved H2 74.3 mm to (101.0, 47.8)
- moved C10 72.0 mm to (3.00, 77.6), turned to 90 degrees
- moved D3 70.5 mm to (5.40, 75.0), turned to 90 degrees
- moved C109 69.6 mm to (12.7, 65.4), turned to 180 degrees
- moved R185 69.5 mm to (1.00, 91.8), turned to 90 degrees
- moved U9 69.3 mm to (10.6, 68.1), turned to 90 degrees
- moved R184 68.1 mm to (1.00, 99.2), turned to 90 degrees
- moved R162 67.7 mm to (54.3, 49.9)
- moved R163 67.7 mm to (62.0, 48.8)
- moved J20 67.7 mm to (57.0, 47.6)
- moved R161 67.7 mm to (53.9, 47.6)
- moved R14 66.8 mm to (14.1, 66.8), turned to 0 degrees
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- renumbered J17 to J5, R194 to R18, U25 to U10, U32 to U4
Connections:
- D32 pad 2: Net-(D32-A) -> unconnected-(D32-A-Pad2)
Routing:
- net 24V: track 224.4 -> 129.0 mm, vias 6 -> 4
- net FLAME_IN: track 67.0 -> 4.69 mm
- net RT_IN: track 58.5 -> 4.75 mm
- net (no net): track 80.9 -> 27.9 mm, vias 6 -> 4
- net SPI_SCK: track 74.6 -> 34.8 mm, vias 4 -> 2
- net PMING_IN: track 50.1 -> 12.1 mm
- net SPI_MOSI: track 69.5 -> 31.6 mm, vias 4 -> 2
- net ANSENS_CS3: track 38.3 -> 4.54 mm
- net ESP32_RX: track 101.3 -> 67.9 mm
- net ESP32_TX: track 101.2 -> 68.7 mm
- net INAIL_IN: track 41.4 -> 12.1 mm
- net FL_PWM: track 46.1 -> 19.1 mm
- net FAN_DEMAND_POS: track 37.5 -> 15.1 mm
- net FAN_ENCODER: track 36.9 -> 14.6 mm
- net FAN_DEMAND_NEG: track 30.9 -> 8.84 mm
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Other:
- outline, holes or cut-outs redrawn
- board text removed: "0/10V"
- board text removed: "AUX RELAYS"
- board text removed: "ESP32 RX"
- board text removed: "ESP32 TX"
- board text removed: "FLAME_1"
- board text removed: "FLAME_2"
- board text removed: "FLS"
- board text removed: "INAIL_1"
- board text removed: "INAIL_2"
- board text removed: "OUT9"
- board text removed: "PMING_1"
- board text removed: "PMING_2"
- board text removed: "RT_1"
- board text removed: "RT_2"
- board text removed: "SBTB"
- board text removed: "SE"
- board text removed: "SF"
- board text removed: "SM"
- board text removed: "SR"
- board text removed: "TL-TF_1"
- board text removed: "TL-TF_2"

Commit message: Schematic design at finish
Parts:
- removed J13: Conn_01x10_Pin, Connector_Phoenix_MC:PhoenixContact_MCV_1,5_10-G-3.81_1x10_P3.81mm_Vertical
- added J1: Conn_01x20_Pin, Connectors:Terminal_Block_3_81_20p_Horizontal, F.Cu at (42.5, 104.8)
- added J2: Jack-DC, Connector_BarrelJack:BarrelJack_GCT_DCJ200-10-A_Horizontal, F.Cu at (63.2, 140.4)
- added K2: G6K-2F-Y-5V, Relays:RELAY_G6K-2F_DC5, F.Cu at (173.6, 62.5)
- added K3: G6K-2F-Y-5V, Relays:RELAY_G6K-2F_DC5, F.Cu at (184.3, 62.7)
- D12: footprint Relays:RELAY_G6K-2F_DC5 -> LED_SMD:LED_RGB_5050-6
- moved J7 66.5 mm to (113.9, 59.4), turned to 90 degrees
- moved D18 49.7 mm to (171.4, 74.8)
- moved Q9 49.7 mm to (166.0, 74.9)
- moved R66 49.7 mm to (168.4, 78.4)
- moved D16 49.7 mm to (163.6, 71.0)
- moved D19 49.7 mm to (172.5, 71.0)
- moved D20 49.7 mm to (180.0, 74.8)
- moved D21 49.7 mm to (181.2, 70.9)
- moved Q10 49.7 mm to (184.1, 74.6)
- moved R164 49.7 mm to (162.6, 79.2)
- moved R165 49.7 mm to (165.0, 78.4)
- moved R175 49.7 mm to (175.2, 78.1)
- moved R176 49.7 mm to (172.7, 77.4)
- moved R177 49.7 mm to (182.1, 78.1)
- moved R178 49.7 mm to (183.8, 78.1)
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Routing:
- net ESP32_TX: track 68.7 -> 55.8 mm, vias 2 -> 1
- net ESP32_RX: track 67.9 -> 55.4 mm, vias 2 -> 1
- net 24V: track 129.0 -> 122.7 mm
- net Net-(D21-A): track 6.59 -> 3.49 mm

Commit message: Layout 90% done
Parts:
- removed C10, C11: 68p/50V, Capacitor_SMD:C_0402_1005Metric
- removed C108, C109: 10p, Capacitor_SMD:C_0402_1005Metric
- removed C12, C19, C8, C9: 100n/25V, Capacitor_SMD:C_0402_1005Metric
- removed D17, D18, D20: RED, LED_SMD:LED_1206_3216Metric
- removed Q22, Q24: BC847BS, Package_TO_SOT_SMD:SOT-363_SC-70-6
- removed R169, R170, R224, R225, R227, R228, R229, R230, R232, R233: 10k, Resistor_SMD:R_0402_1005Metric
- removed R186, R187: 100k, Resistor_SMD:R_0603_1608Metric
- removed R222, R223, R226, R231: 4k7/1%, Resistor_SMD:R_0402_1005Metric
- removed U3, U5, U8, U9: BU4S66G2-TR, Package_TO_SOT_SMD:SOT-23-5
- removed U6: MCP4822, Package_SO:SOIC-8_3.9x4.9mm_P1.27mm
- removed U7: TLV272IS-13, Package_SO:VSSOP-8_3x3mm_P0.65mm
- added C22: 100n/50V, Capacitor_SMD:C_0402_1005Metric, F.Cu at (45.6, 141.1)
- added D13: LED_RGB, LED_SMD:LED_RGB_5050-6, F.Cu at (112.2, 90.8)
- added D14: RED, LED_SMD:LED_0603_1608Metric, F.Cu at (68.0, 56.3)
- added D15: RED, LED_SMD:LED_0603_1608Metric, F.Cu at (57.9, 64.2)
- added G***: LOGO, LOGO, F.Cu at (50.4, 146.5)
- added K4: G6K-2F-Y-24V, Relays:RELAY_G6K-2F_DC5, F.Cu at (51.5, 60.9)
- added Q1: BC847BS, Package_TO_SOT_SMD:SOT-363_SC-70-6, F.Cu at (109.7, 101.3)
- added Q2: BC847BS, Package_TO_SOT_SMD:SOT-363_SC-70-6, F.Cu at (113.6, 105.6)
- added Q3: BC847BS, Package_TO_SOT_SMD:SOT-363_SC-70-6, F.Cu at (58.8, 61.1)
- added R41: 2k2, Resistor_SMD:R_0603_1608Metric, F.Cu at (106.5, 104.5)
- added R42: 10k, Resistor_SMD:R_0603_1608Metric, F.Cu at (106.5, 102.7)
- added R43: 10k, Resistor_SMD:R_0603_1608Metric, F.Cu at (108.0, 95.1)
- added R44: 10k, Resistor_SMD:R_0603_1608Metric, F.Cu at (106.3, 95.1)
- added R45: 10k, Resistor_SMD:R_0603_1608Metric, F.Cu at (116.2, 92.4)
- added R46: 0R, Resistor_SMD:R_0603_1608Metric, F.Cu at (108.5, 91.0)
- added R48: 2k2, Resistor_SMD:R_0603_1608Metric, F.Cu at (112.0, 102.0)
- added R49: 10k, Resistor_SMD:R_0603_1608Metric, F.Cu at (113.7, 102.0)
- added R50: 2k2, Resistor_SMD:R_0603_1608Metric, F.Cu at (109.8, 106.0)
- added R51: 10k, Resistor_SMD:R_0603_1608Metric, F.Cu at (110.6, 108.4)
- C3, C5: value 100n/25V -> 68p/50V
- D12: value LED_RGBA -> RED; footprint LED_SMD:LED_RGB_5050-6 -> LED_SMD:LED_0603_1608Metric
- D16, D19, D21: value US1A -> BAT46W; footprint Diode_SMD:D_SMA -> Diode_SMD:D_SOD-123
- D3: value SMAJ12A -> RED; footprint Diode_SMD:D_SMA -> LED_SMD:LED_0603_1608Metric
- D4: value SMAJ12A -> BAT46W; footprint Diode_SMD:D_SMA -> Diode_SMD:D_SOD-123
- K1, K2, K3: value G6K-2F-Y-5V -> G6K-2F-Y-24V
- R10: value 0R/1% -> 10k
- R11: value 2k2/1% -> 10k
- R113: footprint Resistor_SMD:R_0603_1608Metric -> Resistor_SMD:R_0402_1005Metric
- R12: value 2k2/1% -> 680R
- R13: value 4k7/1% -> 680R; footprint Resistor_SMD:R_0603_1608Metric -> Resistor_SMD:R_0402_1005Metric
- R14: value 4k7/1% -> 0R/1%
- R38, R39, R40, R82, R83: footprint Resistor_SMD:R_0603_1608Metric -> Resistor_SMD:R_1206_3216Metric
- R8, R9: value 0R/1% -> 2k2
- moved R8 210.7 mm to (196.0, 62.8), turned to 0 degrees
- moved R9 209.7 mm to (196.0, 65.4), turned to 0 degrees
- moved R15 184.9 mm to (117.8, 53.0), turned to 180 degrees
- moved R20 182.9 mm to (116.6, 65.4), turned to 180 degrees
- moved C16 181.1 mm to (118.9, 65.8), turned to -90 degrees
- moved R17 177.4 mm to (111.0, 62.9), turned to 90 degrees
- moved C17 176.9 mm to (114.4, 65.6), turned to -90 degrees
- moved R16 176.7 mm to (109.3, 55.3), turned to -90 degrees
- moved C14 175.0 mm to (111.7, 55.9), turned to 90 degrees
- moved C15 171.4 mm to (109.2, 64.1), turned to -90 degrees
- moved R26 170.3 mm to (97.8, 52.5), turned to -90 degrees
- moved C20 166.9 mm to (100.3, 55.0), turned to 90 degrees
- moved R23 166.4 mm to (96.1, 52.5), turned to -90 degrees
- moved C21 166.4 mm to (99.2, 55.0), turned to 90 degrees
- moved C18 165.4 mm to (100.8, 58.5)
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Connections:
- C106 pad 2: Net-(C106-Pad2) -> SM
- C107 pad 2: Net-(C107-Pad2) -> SR
- C14 pad 1: 5V_USB -> 5V_USB'
- C15 pad 1: 5V_USB -> 5V_USB'
- C17 pad 1: 5V_USB -> 5V_USB'
- C20 pad 1: 5V_USB -> 5V_USB'
- C21 pad 1: 5V_USB -> 5V_USB'
- C3 pad 1: 11V -> AUXUART_RX
- C5 pad 1: 11V -> AUXUART_TX
- C7 pad 1: 3V3 -> 5V_USB'
- D12 pad 1: Net-(D12-RK) -> Net-(D12-K)
- D12 pad 2: Net-(D12-GK) -> Net-(D12-A)
- D3 pad 1: SB-TB -> Net-(D3-K)
- D3 pad 2: GND -> Net-(D3-A)
- D32 pad 2: unconnected-(D32-A-Pad2) -> Net-(D32-A)
- D4 pad 1: SE -> 24V
- D4 pad 2: GND -> Net-(D4-A)
- J1 pad 10: unconnected-(J1-Pin_10-Pad10) -> GND
- J1 pad 11: unconnected-(J1-Pin_11-Pad11) -> SM
- J1 pad 12: unconnected-(J1-Pin_12-Pad12) -> GND
- J1 pad 13: unconnected-(J1-Pin_13-Pad13) -> AUXUART_RX
- J1 pad 14: unconnected-(J1-Pin_14-Pad14) -> AUXUART_TX
- J1 pad 15: unconnected-(J1-Pin_15-Pad15) -> RS485_A
- J1 pad 16: unconnected-(J1-Pin_16-Pad16) -> RS485_B
- J1 pad 17: unconnected-(J1-Pin_17-Pad17) -> CANL
- J1 pad 18: unconnected-(J1-Pin_18-Pad18) -> CANH
- J1 pad 19: unconnected-(J1-Pin_19-Pad19) -> GND
- J1 pad 20: unconnected-(J1-Pin_20-Pad20) -> 24V
- J1 pad 3: CANH -> unconnected-(J1-Pin_3-Pad3)
- J1 pad 4: CANL -> unconnected-(J1-Pin_4-Pad4)
- J1 pad 5: RS485_B -> unconnected-(J1-Pin_5-Pad5)
- J1 pad 6: RS485_A -> unconnected-(J1-Pin_6-Pad6)
- J1 pad 7: ESP32_RX -> unconnected-(J1-Pin_7-Pad7)
- J1 pad 8: ESP32_TX -> unconnected-(J1-Pin_8-Pad8)
- J1 pad 9: unconnected-(J1-Pin_9-Pad9) -> SR
- J24 pad 5: Net-(J24-Pin_5) -> unconnected-(J24-Pin_5-Pad5)
- J7 pad A4: 5V_USB -> 5V_USB'
- J7 pad A9: 5V_USB -> 5V_USB'
- J7 pad B4: 5V_USB -> 5V_USB'
- J7 pad B9: 5V_USB -> 5V_USB'
- J8 pad 2: unconnected-(J8-Pin_2-Pad2) -> USB_TX
- J8 pad 3: unconnected-(J8-Pin_3-Pad3) -> USB_RX
- J8 pad 4: unconnected-(J8-Pin_4-Pad4) -> 5V_USB'
- Q8 pad 3: Net-(D18-K) -> Net-(D12-K)
- Q9 pad 3: Net-(D17-K) -> Net-(D3-K)
- R10 pad 1: GND -> Net-(Q3B-B2)
- R10 pad 2: Net-(U6-~{LDAC}) -> GND
- R11 pad 1: Net-(U7A--) -> Net-(Q3A-B1)
- R12 pad 1: Net-(U7B--) -> 3V3
- R12 pad 2: GND -> Net-(D15-A)
- R122 pad 2: ESP32_TX -> AUXUART_TX
- R13 pad 1: Net-(C108-Pad2) -> Net-(D32-A)
- R13 pad 2: Net-(U7A--) -> STATUS_LED_3
- R14 pad 1: Net-(C109-Pad2) -> Net-(U12-3V3OUT)
- R14 pad 2: Net-(U7B--) -> Net-(U12-VCCIO)
- R148 pad 2: ESP32_RX -> AUXUART_RX
- R20 pad 2: 5V_USB -> 5V_USB'
- R23 pad 1: 5V_USB -> 5V_USB'
- R26 pad 1: 5V_USB -> 5V_USB'
- R3 pad 1: Net-(C106-Pad2) -> SM
- R38 pad 1: Net-(D12-BK) -> Net-(Q1B-C2)
- R38 pad 2: B_LED -> Net-(D13-GK)
- R39 pad 1: Net-(D12-GK) -> Net-(Q2A-C1)
- R39 pad 2: G_LED -> Net-(D13-BK)
- R40 pad 1: Net-(D12-RK) -> Net-(Q1A-C1)
- R40 pad 2: R_LED -> Net-(D13-RK)
- R6 pad 1: Net-(C107-Pad2) -> SR
- R64 pad 2: Net-(D17-A) -> Net-(D3-A)
- R69 pad 2: Net-(D18-A) -> Net-(D12-A)
- R8 pad 1: Net-(U6-VA) -> Net-(Q3A-B1)
- R8 pad 2: Net-(U7A-+) -> PMING_IN
- R9 pad 1: Net-(U6-VB) -> Net-(Q3B-B2)
- R9 pad 2: Net-(U7B-+) -> PMING_IN
- U1 pad 15: ADC1_IN10 -> unconnected-(U1-PC0-Pad15)
- U1 pad 30: ANSENS_CS4 -> unconnected-(U1-PA5-Pad30)
- U1 pad 31: EN_WPT-WPS -> unconnected-(U1-PA6-Pad31)
- U1 pad 32: EN_SS-SC -> unconnected-(U1-PA7-Pad32)
- U1 pad 33: ANSENS_CS3 -> unconnected-(U1-PC4-Pad33)
- U1 pad 34: EN_SF -> unconnected-(U1-PC5-Pad34)
- U1 pad 35: EN_0-10V -> unconnected-(U1-PB0-Pad35)
- U1 pad 39: ANSENS_CS2 -> unconnected-(U1-PE8-Pad39)
- U1 pad 40: EN_SE -> unconnected-(U1-PE9-Pad40)
- U1 pad 41: EN_SB-TB -> unconnected-(U1-PE10-Pad41)
- U1 pad 43: EN_SR -> unconnected-(U1-PE12-Pad43)
- U1 pad 44: EN_SM -> unconnected-(U1-PE13-Pad44)
- U1 pad 45: FL_PWM -> unconnected-(U1-PE14-Pad45)
- U1 pad 64: unconnected-(U1-PC7-Pad64) -> B_LED
- U1 pad 65: unconnected-(U1-PC8-Pad65) -> G_LED
- U1 pad 66: unconnected-(U1-PC9-Pad66) -> R_LED
- U1 pad 7: FAN_DEMAND_NEG -> unconnected-(U1-PC13-Pad7)
- U1 pad 78: unconnected-(U1-PC10-Pad78) -> STATUS3_LED
- U1 pad 79: OUT7_STATUS -> STATUS2_LED
- U1 pad 80: OUT6_STATUS -> STATUS1_LED
- U1 pad 81: OUT5_STATUS -> BATTERY_LED
- U1 pad 82: OUT4_STATUS -> GRID_LED
- U1 pad 83: OUT3_STATUS -> DIPSW_6
- U1 pad 84: OUT2_STATUS -> DIPSW_5
- U1 pad 85: OUT1_STATUS -> DIPSW_4
- U1 pad 86: OUT8_STATUS -> DIPSW_3
- U1 pad 87: OUT9_STATUS -> DIPSW_2
- U1 pad 88: OUT0_STATUS -> DIPSW_1
- U1 pad 95: FAN_DEMAND_POS -> unconnected-(U1-PB8-Pad95)
- U1 pad 96: FAN_ENCODER -> unconnected-(U1-PB9-Pad96)
- U1 pad 97: RLY_AUX1 -> unconnected-(U1-PE0-Pad97)
- U1 pad 98: RLY_AUX2 -> unconnected-(U1-PE1-Pad98)
- U11 pad 1: 5V_USB -> 5V_USB'
- U11 pad 8: 5V_USB -> 5V_USB'
- U12 pad 20: 5V_USB -> 5V_USB'
- U12 pad 4: 3V3 -> Net-(U12-VCCIO)
- U24 pad 1: Net-(C106-Pad2) -> SM
- U24 pad 7: Net-(C107-Pad2) -> SR
Routing:
- net 3V3: track 61.2 -> 247.9 mm, vias 18 -> 12
- net 5V_USB': track 0.00 -> 106.8 mm
- net STATUS3_LED: track 0.00 -> 104.7 mm
- net STATUS2_LED: track 0.00 -> 96.3 mm
- net STATUS1_LED: track 0.00 -> 86.8 mm
- net Net-(U1-PA2): track 2.21 -> 80.9 mm
- net BATTERY_LED: track 0.00 -> 77.6 mm
- net Net-(U1-PA3): track 2.28 -> 79.7 mm
- net 5V: track 177.2 -> 249.4 mm, vias 7 -> 8
- net 11V: track 152.6 -> 85.4 mm, vias 11 -> 0
- net GRID_LED: track 0.00 -> 66.6 mm
- net ESP32_TX: track 55.8 -> 0.00 mm, vias 1 -> 0
- net ESP32_RX: track 55.4 -> 0.00 mm, vias 1 -> 0
- net DIPSW_1: track 0.00 -> 44.2 mm
- net DIPSW_2: track 0.00 -> 43.8 mm
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- added copper zone on B.Cu, net GND
- added copper zone on F.Cu, net GND
Other:
- board size 172.1 x 119.7 mm -> 87 x 103.7 mm
- copper layers 4 -> 2
- board text added: "0.1"
- board text removed: "0.2"
- board text removed: "CANH"
- board text removed: "CANL"
- board text removed: "RS485 A"
- board text removed: "RS485 B"
- board text removed: "RTB"

Commit message: Gate finalized! PCB ordered
Parts:
- added H5: MountingHole, MountingHole:MountingHole_2.2mm_M2, F.Cu at (118.3, 117.9)
- added H6: MountingHole, MountingHole:MountingHole_2.2mm_M2, F.Cu at (118.3, 136.3)
- R10, R66, R68, R71: value 10k -> 100k
- R12, R64, R69, R72: value 680R -> 22k
- R65, R67, R70, R9: value 2k2 -> 10k
- moved R9 134.3 mm to (62.0, 56.9)
- moved R8 134.2 mm to (62.0, 55.1)
- moved Q10 125.7 mm to (58.5, 69.8), turned to 0 degrees
- moved R71 125.4 mm to (62.2, 66.5), turned to 0 degrees
- moved R70 123.6 mm to (62.2, 68.1), turned to 0 degrees
- moved R72 122.9 mm to (57.6, 72.9)
- moved R178 121.9 mm to (62.2, 69.7), turned to 0 degrees
- moved R177 120.1 mm to (62.2, 71.4), turned to 0 degrees
- moved R68 110.5 mm to (62.2, 75.1), turned to 0 degrees
- moved Q8 110.1 mm to (58.5, 80.9), turned to 0 degrees
- moved R67 108.7 mm to (62.2, 76.8), turned to 0 degrees
- moved R175 106.7 mm to (62.2, 78.6), turned to 0 degrees
- moved R69 105.7 mm to (57.7, 84.0)
- moved R176 104.0 mm to (62.2, 80.3), turned to 0 degrees
- moved G*** 88.4 mm to (88.1, 66.5)
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Connections:
- C22 pad 1: 24V -> Vin
- C52 pad 1: Net-(C52-Pad1) -> Vin
- C54 pad 1: Net-(C52-Pad1) -> Vin
- D16 pad 1: 24V -> Vin
- D19 pad 1: 24V -> Vin
- D21 pad 1: 24V -> Vin
- D4 pad 1: 24V -> Vin
- F1 pad 2: Net-(C52-Pad1) -> Vin
- J1 pad 1: unconnected-(J1-Pin_1-Pad1) -> RLY4_B
- J1 pad 2: unconnected-(J1-Pin_2-Pad2) -> RLY4_A
- J1 pad 20: 24V -> Vin
- J1 pad 3: unconnected-(J1-Pin_3-Pad3) -> RLY3_B
- J1 pad 4: unconnected-(J1-Pin_4-Pad4) -> RLY3_A
- J1 pad 5: unconnected-(J1-Pin_5-Pad5) -> RLY2_B
- J1 pad 6: unconnected-(J1-Pin_6-Pad6) -> RLY2_A
- J1 pad 7: unconnected-(J1-Pin_7-Pad7) -> RLY1_B
- J1 pad 8: unconnected-(J1-Pin_8-Pad8) -> RLY1_A
- J8 pad 2: USB_TX -> USB_TX_OUT
- J8 pad 3: USB_RX -> USB_RX_OUT
- K1 pad 1: 24V -> Vin
- K1 pad 3: RLY1_B -> RLY1_A
- K1 pad 4: RLY1_A -> RLY1_B
- K2 pad 1: 24V -> Vin
- K2 pad 2: RLY2_A -> unconnected-(K2-Pad2)
- K2 pad 3: RLY2_B -> RLY2_A
- K2 pad 4: unconnected-(K2-Pad4) -> RLY2_B
- K3 pad 1: 24V -> Vin
- K3 pad 2: RLY3_A -> unconnected-(K3-Pad2)
- K3 pad 3: RLY3_B -> RLY3_A
- K3 pad 4: unconnected-(K3-Pad4) -> RLY3_B
- K4 pad 1: 24V -> Vin
- K4 pad 2: RLY3_A -> unconnected-(K4-Pad2)
- K4 pad 3: RLY3_B -> RLY4_A
- K4 pad 4: unconnected-(K4-Pad4) -> RLY4_B
- L4 pad 1: Net-(C52-Pad1) -> Vin
- R12 pad 1: 3V3 -> Vin
- R22 pad 2: 5V_USB -> 5V_USB'
- R24 pad 2: USB_RX -> USB_RX_OUT
- R25 pad 2: USB_TX -> USB_TX_OUT
- R64 pad 1: 3V3 -> Vin
- R69 pad 1: 3V3 -> Vin
- R72 pad 1: 3V3 -> Vin
- R8 pad 2: PMING_IN -> RT_IN
- R9 pad 2: PMING_IN -> RT_IN
- U1 pad 1: FLAME_IN -> unconnected-(U1-PE2-Pad1)
Routing:
- net Vin: track 0.00 -> 189.1 mm
- net 24V: track 139.4 -> 42.1 mm
- net SPI_SCK: track 1.88 -> 79.2 mm, vias 0 -> 2
- net SPI_MOSI: track 1.74 -> 75.6 mm, vias 0 -> 2
- net SPI_MISO: track 3.10 -> 62.9 mm
- net I2C_SDA: track 1.47 -> 59.8 mm
- net I2C_SCK: track 12.2 -> 69.2 mm
- net 3V3: track 247.9 -> 301.7 mm, vias 12 -> 8
- net 5V: track 249.4 -> 214.9 mm, vias 8 -> 2
- net RT_IN: track 42.0 -> 68.4 mm
- net Net-(Q9A-B1): track 0.00 -> 22.5 mm
- net Net-(Q9B-B2): track 0.00 -> 22.5 mm
- net RLY4_A: track 0.00 -> 20.7 mm
- net Net-(C52-Pad1): track 16.0 -> 0.00 mm
- net RLY3_A: track 0.00 -> 15.8 mm
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