File: HilBox_MCU.kicad_sch (KiCad schematic)
At the start: 53 parts, among them J11 Conn_01x03_Pin, J20 Conn_01x04_Pin, J24 Conn_01x06_Pin, U1 STM32F407VGTx, Y1 20MHz

Commit message: Modification in half of target
Parts:
- removed R126: 220R, Resistor_SMD:R_0402_1005Metric, symbol Device:R
- D32: value YELLOW -> RED
- D33: value PURPLE -> RED
- D34: value AMBER -> RED
- R125, R166: value 220R -> 680R; JLC_PN C1091 -> C25177
Changed lines of the file:
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@@
 			)
 		)
-		(property "Value" "AMBER"
+		(property "Value" "RED"
 			(at 33.782 160.528 90)
 			(effects
@@
 			)
 		)
-		(property "Value" "220R"
+		(property "Value" "680R"
 			(at 28.194 147.32 90)
 			(effects
@@
 			)
 		)
-		(property "JLC_PN" "C1091"
+		(property "JLC_PN" "C25177"
 			(at 30.48 149.86 90)
 			(effects
@@
 			)
 		)
-		(property "Value" "220R"
+		(property "Value" "680R"
 			(at 14.224 147.32 90)
 			(effects
@@
 			)
 		)
-		(property "JLC_PN" "C1091"
+		(property "JLC_PN" "C25177"
 			(at 16.51 149.86 90)
 			(effects
@@
 	)
 	(symbol
-		(lib_id "Device:R")
-		(at 43.18 149.86 180)
-		(unit 1)
-		(exclude_from_sim no)
-		(in_bom yes)
-		(on_board yes)
-		(dnp no)
-		(property "Reference" "R126"
-			(at 43.18 147.32 90)
-			(effects
-				(font
-					(size 1.27 1.27)
-				)
-				(justify left)
-			)
-		)
-		(property "Value" "220R"
-			(at 40.894 147.32 90)
-			(effects
-				(font
-					(size 1.27 1.27)
-				)
-				(justify left)
-			)
-		)
-		(property "Footprint" "Resistor_SMD:R_0402_1005Metric"
-			(at 44.958 149.86 90)
-			(effects
-				(font
-					(size 1.27 1.27)
-				)
-				(hide yes)
-			)
-		)
-		(property "Datasheet" "~"
-			(at 43.18 149.86 0)
-			(effects
-				(font
-					(size 1.27 1.27)
-				)
-				(hide yes)
-			)
-		)
-		(property "Description" "Resistor"
-			(at 43.18 149.86 0)
-			(effects
-				(font
-					(size 1.27 1.27)
-				)
-				(hide yes)
-			)
-		)
-		(property "JLC_PN" "C1091"
-			(at 43.18 149.86 90)
-			(effects
-				(font
-					(size 1.27 1.27)
-				)
-				(hide yes)
-			)
-		)
-		(property "JLC_PCB" ""
-			(at 43.18 149.86 0)
-			(effects
-				(font
-					(size 1.27 1.27)
-				)
-				(hide yes)
-			)
-		)
-		(pin "2"
-		)
-		(pin "1"
-		)
-		(instances
-			(project "HilBox"
-				(path "/c950b3bb-3e52-4d0d-8bbf-240895efa80b/80d7f8d4-2eff-419a-a5a7-9b0e853e9191"
-					(reference "R126")
-					(unit 1)
-				)
-			)
-		)
-	)
-	(symbol
 		(lib_id "power:GND")
 		(at 31.75 120.65 0)
@@
 			)
 		)
-		(property "Value" "YELLOW"
+		(property "Value" "RED"
 			(at 46.482 160.528 90)
 			(effects
@@
 			)
 		)
-		(property "Value" "PURPLE"
+		(property "Value" "RED"
 			(at 19.812 160.528 90)
 			(effects

Commit message: Layout 90% done
Parts:
- removed R169, R170: 10k, Resistor_SMD:R_0402_1005Metric, symbol Device:R
- added R13: 680R, Resistor_SMD:R_0402_1005Metric, symbol Device:R
Connections:
- net STATUS_LED_3: now also R13.2
- net B_LED: now reaches U1.64 (PC7)
- net G_LED: now reaches U1.65 (PC8)
- net R_LED: now reaches U1.66 (PC9)
- net STATUS3_LED: now reaches U1.78 (PC10)
- net at D32.2 (A): now also R13.1
- net ADC1_IN10: no longer names the net of U1.15 (PC0)
- net ANSENS_CS2: no longer names the net of U1.39 (PE8)
- net ANSENS_CS3: no longer names the net of U1.33 (PC4)
- net ANSENS_CS4: no longer names the net of U1.30 (PA5)
- net EN_0-10V: no longer names the net of U1.35 (PB0)
- net EN_SB-TB: no longer names the net of U1.41 (PE10)
- net EN_SE: no longer names the net of U1.40 (PE9)
- net EN_SF: no longer names the net of U1.34 (PC5)
- net EN_SM: no longer names the net of U1.44 (PE13)
- net EN_SR: no longer names the net of U1.43 (PE12)
- net EN_SS-SC: no longer names the net of U1.32 (PA7)
- net EN_WPT-WPS: no longer names the net of U1.31 (PA6)
- net ESP32_RX renamed AUXUART_RX
- net ESP32_TX renamed AUXUART_TX
- net FAN_DEMAND_NEG: no longer names the net of U1.7 (PC13)
- net FAN_DEMAND_POS: no longer names the net of U1.95 (PB8)
- net FAN_ENCODER: no longer names the net of U1.96 (PB9)
- net FL_PWM: no longer names the net of U1.45 (PE14)
- net OUT0_STATUS renamed DIPSW_1
- net OUT1_STATUS renamed DIPSW_4
- net OUT2_STATUS renamed DIPSW_5
- net OUT3_STATUS renamed DIPSW_6
- net OUT4_STATUS renamed GRID_LED
- net OUT5_STATUS renamed BATTERY_LED
- net OUT6_STATUS renamed STATUS1_LED
- net OUT7_STATUS renamed STATUS2_LED
- net OUT8_STATUS renamed DIPSW_3
- net OUT9_STATUS renamed DIPSW_2
- net RLY_AUX1: no longer names the net of U1.97 (PE0)
- net RLY_AUX2: no longer names the net of U1.98 (PE1)

Commit message: Gate finalized! PCB ordered
Connections:
- net FLAME_IN: no longer names the net of U1.1 (PE2)
Changed lines of the file:
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@@
-	(wire
-		(pts
-			(xy 71.12 73.66) (xy 91.44 73.66)
-		)
-		(stroke
-			(width 0)
-			(type default)
-		)
-	)
 	(wire
 		(pts
@@
 			(effects
 				(font
-					(size 1.27 1.27)
-				)
-				(justify right)
-				(hide yes)
-			)
-		)
-	)
-	(global_label "FLAME_IN"
-		(shape input)
-		(at 71.12 73.66 180)
-		(fields_autoplaced yes)
-		(effects
-			(font
-				(size 1.27 1.27)
-			)
-			(justify right)
-		)
-		(property "Intersheetrefs" "${INTERSHEET_REFS}"
-			(at 59.4262 73.66 0)
-			(effects
-				(font
